Commit message: update launch and gen urdf file

File: urdf/hbot.urdf (robot description, URDF)
Before this commit: robot hbot, 4 links, 3 joints
Links:
- added link left_wheel_link; visual cylinder length=0.025 radius=0.0325
- added link right_wheel_link; visual cylinder length=0.025 radius=0.0325
- link base_link: geometry visual box size=0.17 0.14 0.08
- link front_caster: geometry visual sphere radius=0.01
Joints:
- added joint left_wheel_joint: type continuous, parent base_link, child left_wheel_link, origin xyz=-0.05 0.10500000000000001 -0.05 rpy=0 0 0, axis 0 1 0
- added joint right_wheel_joint: type continuous, parent base_link, child right_wheel_link, origin xyz=-0.05 -0.10500000000000001 -0.05 rpy=0 0 0, axis 0 1 0
- joint base_joint: child base_footprint -> base_link; origin xyz=0 0 ${-(wheel_radius+wheel_zoff)} rpy=0 0 0 -> xyz=0 0 0.0825 rpy=0 0 0; parent base_link -> base_footprint
- joint front_caster_joint: origin xyz=${caster_xoff} 0.0 ${-wheel_zoff-caster_radius} rpy=0 0 0 -> xyz=0.07 0.0 -0.060000000000000005 rpy=0 0 0
- joint lidar_joint: origin xyz=0 0 ${base_height/2+0.015} rpy=0 0 0 -> xyz=0 0 0.055 rpy=0 0 0

Commit message: fix: change laser frame id

File: urdf/hbot.urdf (robot description, URDF)
Before this commit: robot hbot, 6 links, 5 joints
Links:
- removed link lidar_link
- added link laser; visual cylinder length=0.025 radius=0.03
Joints:
- joint lidar_joint: child lidar_link -> laser

File: urdf/hbot.urdf.xacro (robot description, xacro)
@@ -71,5 +71,5 @@
   </joint>
   <!-- Lidar -->
-  <link name="lidar_link">
+  <link name="laser">
     <visual>
       <geometry>
@@ -83,5 +83,5 @@
   <joint name="lidar_joint" type="fixed">
     <parent link="base_link"/>
-    <child link="lidar_link"/>
+    <child link="laser"/>
     <origin xyz="0 0 ${base_height/2+0.015}" rpy="0 0 0"/>
   </joint>

Commit message: fix: add inertials, material files. Fix urdf xacro to load to gazebo

File: urdf/hbot.urdf (robot description, URDF)
Before this commit: robot hbot, 6 links, 5 joints
Links:
- link base_link: mass None -> 0.5; geometry collision box size=0.17 0.14 0.08; visual box size=0.17 0.14 0.08
- link front_caster: mass None -> 0.001; geometry collision sphere radius=0.01; visual sphere radius=0.01
- link laser: mass None -> 0.001; geometry collision cylinder length=0.025 radius=0.03; visual cylinder length=0.025 radius=0.03
- link left_wheel_link: mass None -> 0.1; geometry collision cylinder length=0.025 radius=0.0325; visual cylinder length=0.025 radius=0.0325
- link right_wheel_link: mass None -> 0.1; geometry collision cylinder length=0.025 radius=0.0325; visual cylinder length=0.025 radius=0.0325
Joints:
- joint front_caster_joint: origin xyz=0.07 0.0 -0.060000000000000005 rpy=0 0 0 -> xyz=0.07 0.0 -0.07250000000000001 rpy=0 0 0

File: urdf/hbot.urdf.xacro (robot description, xacro)
@@ -1,4 +1,6 @@
 <?xml version="1.0" ?>
 <robot name="hbot" xmlns:xacro="http://ros.org/wiki/xacro">
+  <xacro:include filename="$(find hbot_description)/urdf/inertials.xacro" />
+  <xacro:include filename="$(find hbot_description)/urdf/materials.xacro" />
   <!-- Define some constants -->
   <xacro:property name="base_width" value="0.14"/>
@@ -12,4 +14,10 @@
   <xacro:property name="caster_radius" value="0.01"/>
   <xacro:property name="caster_xoff" value="0.07"/>
+  <link name="base_footprint"/>
+  <joint name="base_joint" type="fixed">
+    <parent link="base_footprint"/>
+    <child link="base_link"/>
+    <origin xyz="0 0 ${(wheel_radius+wheel_zoff)}" rpy="0 0 0"/>
+  </joint>
   <link name="base_link">
     <visual>
@@ -21,11 +29,14 @@
       </material>
     </visual>
+    <collision>
+      <geometry>
+        <box size="${base_length} ${base_width} ${base_height}"/>
+      </geometry>
+    </collision>
+    <xacro:solid_cuboid_inertial
+      rpy="0 0 0" xyz="0 0 0" mass="0.5"
+      x="${base_length}" y="${base_width}" z="${base_height}"
+    />
   </link>
-  <link name="base_footprint"/>
-  <joint name="base_joint" type="fixed">
-    <parent link="base_footprint"/>
-    <child link="base_link"/>
-    <origin xyz="0 0 ${(wheel_radius+wheel_zoff)}" rpy="0 0 0"/>
-  </joint>
   <!-- Wheel -->
   <xacro:macro name="wheel" params="prefix x_reflect y_reflect">
@@ -43,4 +54,17 @@
         </material>
       </visual>
+      <collision>
+        <origin xyz="0 0 0" rpy="${pi/2} 0 0"/>
+        <geometry>
+          <cylinder radius="${wheel_radius}" length="${wheel_width}"/>
+        </geometry>
+      </collision>
+      <xacro:solid_cylinder_inertial
+        rpy="0 0 0"
+        xyz="0 0 0"
+        mass="0.1"
+        radius="${wheel_radius}"
+        length="${wheel_width}"
+      />
     </link>
     <joint name="${prefix}_joint" type="continuous">
@@ -57,5 +81,4 @@
     <visual>
       <geometry>
-        <!-- <sphere radius="${(wheel_radius+wheel_zoff-(base_height/2))}"/> -->
         <sphere radius="${caster_radius}"/>
       </geometry>
@@ -64,9 +87,15 @@
       </material>
     </visual>
+    <collision>
+      <geometry>
+        <sphere radius="${caster_radius}"/>
+      </geometry>
+    </collision>
+    <xacro:null_inertial/>
   </link>
   <joint name="front_caster_joint" type="fixed">
     <parent link="base_link"/>
     <child link="front_caster"/>
-    <origin xyz="${caster_xoff} 0.0 ${-wheel_zoff-caster_radius}" rpy="0 0 0"/>
+    <origin xyz="${caster_xoff} 0.0 ${-wheel_zoff-wheel_radius+caster_radius}" rpy="0 0 0"/>
   </joint>
   <!-- Lidar -->
@@ -80,4 +109,10 @@
       </material>
     </visual>
+    <collision>
+      <geometry>
+        <cylinder radius="0.03" length="0.025"/>
+      </geometry>
+    </collision>
+    <xacro:null_inertial/>
   </link>
   <joint name="lidar_joint" type="fixed">

Commit message: Fix: fix hbot model, add lidar and diff_drive

File: urdf/hbot.urdf (robot description, URDF)
Before this commit: robot hbot, 6 links, 5 joints
Links:
- link base_link: geometry collision box size=0.17 0.14 0.12; visual box size=0.17 0.14 0.12
Joints:
- joint left_wheel_joint: origin xyz=-0.05 0.10500000000000001 -0.05 rpy=0 0 0 -> xyz=-0.05 0.085 -0.05 rpy=0 0 0
- joint lidar_joint: origin xyz=0 0 0.055 rpy=0 0 0 -> xyz=0 0 0.075 rpy=0 0 0
- joint right_wheel_joint: origin xyz=-0.05 -0.10500000000000001 -0.05 rpy=0 0 0 -> xyz=-0.05 -0.085 -0.05 rpy=0 0 0

File: urdf/hbot.urdf.xacro (robot description, xacro)
@@ -5,9 +5,9 @@
   <!-- Define some constants -->
   <xacro:property name="base_width" value="0.14"/>
-  <xacro:property name="base_height" value="0.08"/>
+  <xacro:property name="base_height" value="0.12"/>
   <xacro:property name="base_length" value="0.17"/>
   <xacro:property name="wheel_radius" value="0.0325"/>
   <xacro:property name="wheel_width" value="0.025"/>
-  <xacro:property name="wheel_ygap" value="0.035"/>
+  <xacro:property name="wheel_ygap" value="0.015"/>
   <xacro:property name="wheel_zoff" value="0.05"/>
   <xacro:property name="wheel_xoff" value="0.05"/>
@@ -39,4 +39,7 @@
     />
   </link>
+  <gazebo reference="base_link">
+    <material>Gazebo/Green</material>
+  </gazebo>
   <!-- Wheel -->
   <xacro:macro name="wheel" params="prefix x_reflect y_reflect">
@@ -74,4 +77,7 @@
       <axis xyz="0 1 0"/>
     </joint>
+    <gazebo reference="${prefix}_link">
+      <material>Gazebo/Black</material>
+    </gazebo>
   </xacro:macro>
   <xacro:wheel prefix="left_wheel" x_reflect="-1" y_reflect="1"/>
@@ -121,3 +127,59 @@
     <origin xyz="0 0 ${base_height/2+0.015}" rpy="0 0 0"/>
   </joint>
+  <gazebo reference="laser">
+    <sensor name="lidar" type="ray">
+      <always_on>true</always_on>
+      <visualize>false</visualize>
+      <update_rate>10</update_rate>
+      <ray>
+        <scan>
+          <horizontal>
+            <samples>360</samples>
+            <resolution>1</resolution>
+            <min_angle>-3.14</min_angle>
+            <max_angle>3.14</max_angle>
+          </horizontal>
+        </scan>
+        <range>
+          <min>0.25</min>
+          <max>6.0</max>
+          <resolution>0.02</resolution>
+        </range>
+        <noise>
+          <type>gaussian</type>
+          <mean>0.0</mean>
+          <stddev>0.01</stddev>
+        </noise>
+      </ray>
+      <plugin name="scan" filename="libgazebo_ros_ray_sensor.so">
+        <ros>
+          <remapping>~/out:=scan</remapping>
+        </ros>
+        <output_type>sensor_msgs/LaserScan</output_type>
+        <frame_name>laser</frame_name>
+      </plugin>
+    </sensor>
+  </gazebo>
+  <gazebo reference="laser">
+    <material>Gazebo/Yellow</material>
+  </gazebo>
+  <gazebo>
+    <plugin name="two_front_wheeled_diff_drive" filename="libgazebo_ros_diff_drive.so">
+      <update_rate>30</update_rate>
+      <left_joint>left_wheel_joint</left_joint>
+      <right_joint>right_wheel_joint</right_joint>
+      <wheel_separation>0.3</wheel_separation>
+      <wheel_diameter>0.1</wheel_diameter>
+      <max_wheel_torque>20</max_wheel_torque>
+      <max_wheel_acceleration>1.0</max_wheel_acceleration>
+      <command_topic>cmd_vel</command_topic>
+      <publish_odom>true</publish_odom>
+      <publish_odom_tf>true</publish_odom_tf>
+      <publish_wheel_tf>true</publish_wheel_tf>
+      <odometry_topic>odom</odometry_topic>
+      <odometry_frame>odom</odometry_frame>
+      <robot_base_frame>base_footprint</robot_base_frame>
+      <odometry_source>1</odometry_source>
+    </plugin>
+  </gazebo>
 </robot>

Commit message: fix orientation of lidar

File: urdf/hbot.urdf (robot description, URDF)
Before this commit: robot hbot, 6 links, 5 joints
Joints:
- joint lidar_joint: origin xyz=0 0 0.075 rpy=0 0 0 -> xyz=0 0 0.075 rpy=0 0 3.14

File: urdf/hbot.urdf.xacro (robot description, xacro)
@@ -125,5 +125,5 @@
     <parent link="base_link"/>
     <child link="laser"/>
-    <origin xyz="0 0 ${base_height/2+0.015}" rpy="0 0 0"/>
+    <origin xyz="0 0 ${base_height/2+0.015}" rpy="0 0 3.14"/>
   </joint>
   <gazebo reference="laser">
